Commit message: Changes for URDF and Stuff

File: description/gazebo_control.xacro (robot description, xacro)
@@ -6,16 +6,17 @@
             <left_joint>left_wheel_joint</left_joint>
             <right_joint>right_wheel_joint</right_joint>
-            <wheel_separation>0.4</wheel_separation>
-            <wheel_radius>0.0762</wheel_radius>
+            <wheel_separation>${wheel_separation}</wheel_separation>
+            <wheel_radius>${wheel_radius}</wheel_radius>
             <!-- Input -->
-            <topic>cmd_vel</topic>
+            <topic>/cmd_vel</topic>
             <!-- Output -->
             <frame_id>odom</frame_id>
             <child_frame_id>base_link</child_frame_id>
-            <odom_topic>odom</odom_topic>
-            <tf_topic>tf</tf_topic>
+            <odom_topic>/odom</odom_topic>
+            <tf_topic>/tf</tf_topic>
+            <odom_publish_frequency>50</odom_publish_frequency>
         </plugin>
         <plugin name="gz::sim::systems::JointStatePublisher" filename="gz-sim-joint-state-publisher-system">
-            <topic>joint_states</topic>
+            <topic>/joint_states</topic>
             <joint_name>left_wheel_joint</joint_name>
             <joint_name>right_wheel_joint</joint_name>

File: description/lidar.xacro (robot description, xacro)
@@ -22,3 +22,27 @@
         </xacro:inertial_cylinder>
     </link>
+    <gazebo reference="laser_frame">
+        <sensor name="gpu_lidar" type="gpu_lidar">
+            <topic>/scan</topic>
+            <gz_frame_id>laser_frame</gz_frame_id>
+            <update_rate>7</update_rate>
+            <always_on>true</always_on>
+            <visualize>true</visualize>
+            <lidar>
+                <scan>
+                    <horizontal>
+                        <samples>720</samples>
+                        <resolution>1</resolution>
+                        <min_angle>-${pi}</min_angle>
+                        <max_angle>${pi}</max_angle>
+                    </horizontal>
+                </scan>
+                <range>
+                    <min>0.1</min>
+                    <max>12.0</max>
+                    <resolution>0.01</resolution>
+                </range>
+            </lidar>
+        </sensor>
+    </gazebo>
 </robot>

File: description/robot_core.xacro (robot description, xacro)
@@ -2,4 +2,8 @@
 <robot xmlns:xacro="http://www.ros.org/wiki/xacro"  name="robot">
     <xacro:include filename="intertial_macros.xacro"/>
+    <!-- Drive-wheel dimensions (meters); separation is center-to-center. -->
+    <xacro:property name="wheel_radius" value="0.0762"/>
+    <xacro:property name="wheel_width" value="0.035306"/>
+    <xacro:property name="wheel_separation" value="0.44"/>
     <material name ="white">
         <color rgba="1 1 1 1" />
@@ -91,5 +95,5 @@
         <parent link="base_link"/>
         <child link="left_wheel"/>
-        <origin xyz="0.05 0.2 -0.0538" rpy="-${pi/2} 0 0"/>
+        <origin xyz="0.05 ${wheel_separation / 2} -0.0538" rpy="-${pi/2} 0 0"/>
         <axis xyz="0 0 1"/>
         <limit effort="5.0" velocity="13.8"/>
@@ -98,5 +102,5 @@
         <visual>
             <geometry>
-                <cylinder length="0.0635" radius="0.0762" />
+                <cylinder length="${wheel_width}" radius="${wheel_radius}" />
             </geometry>
             <material name="blue"/>
@@ -104,8 +108,8 @@
         <collision>
             <geometry>
-                <sphere radius="0.0762" />
-            </geometry>
-        </collision>
-        <xacro:inertial_cylinder mass="0.9" length="0.0635" radius="0.0762">
+                <cylinder length="${wheel_width}" radius="${wheel_radius}" />
+            </geometry>
+        </collision>
+        <xacro:inertial_cylinder mass="0.9" length="${wheel_width}" radius="${wheel_radius}">
             <origin xyz="0 0 0" rpy="0 0 0"/>
         </xacro:inertial_cylinder>
@@ -115,5 +119,5 @@
         <parent link="base_link"/>
         <child link="right_wheel"/>
-        <origin xyz="0.05 -0.2 -0.0538" rpy="${pi/2} 0 0"/>
+        <origin xyz="0.05 -${wheel_separation / 2} -0.0538" rpy="${pi/2} 0 0"/>
         <axis xyz="0 0 -1"/>
         <limit effort="5.0" velocity="13.8"/>
@@ -122,5 +126,5 @@
         <visual>
             <geometry>
-                <cylinder length="0.0635" radius="0.0762" />
+                <cylinder length="${wheel_width}" radius="${wheel_radius}" />
             </geometry>
             <material name="blue"/>
@@ -128,8 +132,8 @@
         <collision>
             <geometry>
-                <sphere radius="0.0762" />
-            </geometry>
-        </collision>
-        <xacro:inertial_cylinder mass="0.9" length="0.0635" radius="0.0762">
+                <cylinder length="${wheel_width}" radius="${wheel_radius}" />
+            </geometry>
+        </collision>
+        <xacro:inertial_cylinder mass="0.9" length="${wheel_width}" radius="${wheel_radius}">
             <origin xyz="0 0 0" rpy="0 0 0"/>
         </xacro:inertial_cylinder>
