Commit message: Changes to arduino sketch

File: description/robot_core.xacro (robot description, xacro)
@@ -19,4 +19,12 @@
     <!-- BASE LINK -->
     <link name="base_link">
+    </link>
+        <!-- BASE_FOOTPRINT -->
+    <joint name="base_footprint_joint" type="fixed">
+        <parent link="base_link"/>
+        <child link="base_footprint"/>
+        <origin xyz="0 0 0" rpy="0 0 0"/>
+    </joint>
+    <link name="base_footprint">
     </link>
     <!-- CHASSIS LINK-->

Commit message: Fixed to work with odom

File: description/robot_core.xacro (robot description, xacro)
@@ -57,5 +57,5 @@
         <child link="left_wheel"/>
         <origin xyz="0.1524 0.2032 -0.0508" rpy="-${pi/2} 0 0"/>
-        <axis xyz="0 0 1"/>
+        <axis xyz="0 0 -1"/>
         <limit effort="5.0" velocity="13.8"/>
     </joint>

Commit message: Changes

File: description/robot_core.xacro (robot description, xacro)
@@ -81,5 +81,5 @@
         <child link="right_wheel"/>
         <origin xyz="0.1524 -0.2032 -0.0508" rpy="${pi/2} 0 0"/>
-        <axis xyz="0 0 1"/>
+        <axis xyz="0 0 -1"/>
         <limit effort="5.0" velocity="13.8"/>
     </joint>

Commit message: Fixed issues

File: description/robot_core.xacro (robot description, xacro)
@@ -57,5 +57,5 @@
         <child link="left_wheel"/>
         <origin xyz="0.1524 0.2032 -0.0508" rpy="-${pi/2} 0 0"/>
-        <axis xyz="0 0 -1"/>
+        <axis xyz="0 0 1"/>
         <limit effort="5.0" velocity="13.8"/>
     </joint>

Commit message: Fixed URDF inconsistensy

File: description/robot_core.xacro (robot description, xacro)
@@ -56,5 +56,5 @@
         <parent link="base_link"/>
         <child link="left_wheel"/>
-        <origin xyz="0.1524 0.2032 -0.0508" rpy="-${pi/2} 0 0"/>
+        <origin xyz="0.1524 0.2604 -0.0508" rpy="-${pi/2} 0 0"/>
         <axis xyz="0 0 1"/>
         <limit effort="5.0" velocity="13.8"/>
@@ -80,5 +80,5 @@
         <parent link="base_link"/>
         <child link="right_wheel"/>
-        <origin xyz="0.1524 -0.2032 -0.0508" rpy="${pi/2} 0 0"/>
+        <origin xyz="0.1524 -0.2604 -0.0508" rpy="${pi/2} 0 0"/>
         <axis xyz="0 0 -1"/>
         <limit effort="5.0" velocity="13.8"/>

Commit message: Lifted the wheels to proper height

File: description/robot_core.xacro (robot description, xacro)
@@ -91,5 +91,5 @@
         <parent link="base_link"/>
         <child link="left_wheel"/>
-        <origin xyz="0.05 0.2 -0.13" rpy="-${pi/2} 0 0"/>
+        <origin xyz="0.05 0.2 -0.0538" rpy="-${pi/2} 0 0"/>
         <axis xyz="0 0 1"/>
         <limit effort="5.0" velocity="13.8"/>
@@ -115,5 +115,5 @@
         <parent link="base_link"/>
         <child link="right_wheel"/>
-        <origin xyz="0.05 -0.2 -0.13" rpy="${pi/2} 0 0"/>
+        <origin xyz="0.05 -0.2 -0.0538" rpy="${pi/2} 0 0"/>
         <axis xyz="0 0 -1"/>
         <limit effort="5.0" velocity="13.8"/>
@@ -139,5 +139,5 @@
         <parent link="chassis"/>
         <child link="caster_wheel_left"/>
-        <origin xyz="0.98 0.28 -0.16" rpy="0 0 0"/>
+        <origin xyz="0.98 0.28 -0.0665" rpy="0 0 0"/>
     </joint>
     <link name="caster_wheel_left">
@@ -165,5 +165,5 @@
         <parent link="chassis"/>
         <child link="caster_wheel_right"/>
-        <origin xyz="0.98 -0.28 -0.16" rpy="0 0 0"/>
+        <origin xyz="0.98 -0.28 -0.0665" rpy="0 0 0"/>
     </joint>
     <link name="caster_wheel_right">
