Commit message: CHanges to navigation

File: description/robot_core.xacro (robot description, xacro)
@@ -39,5 +39,5 @@
         </collision>
     </xacro:macro>
-    <!-- BASE LINK -->
+    <!-- BASE LINK planar origin is the drive-wheel axle midpoint. -->
     <link name="base_link">
     </link>
@@ -54,5 +54,7 @@
         <parent link="base_link"/>
         <child link= "chassis"/>
-        <origin xyz="-0.1 0 0"/>
+        <!-- Preserve the physical chassis pose after moving base_link 5 cm
+             forward from its legacy location onto the drive axle. -->
+        <origin xyz="-0.15 0 0"/>
     </joint>
     <link name="chassis">
@@ -95,5 +97,5 @@
         <parent link="base_link"/>
         <child link="left_wheel"/>
-        <origin xyz="0.05 ${wheel_separation / 2} -0.0538" rpy="-${pi/2} 0 0"/>
+        <origin xyz="0 ${wheel_separation / 2} -0.0538" rpy="-${pi/2} 0 0"/>
         <axis xyz="0 0 1"/>
         <limit effort="5.0" velocity="13.8"/>
@@ -119,5 +121,5 @@
         <parent link="base_link"/>
         <child link="right_wheel"/>
-        <origin xyz="0.05 -${wheel_separation / 2} -0.0538" rpy="${pi/2} 0 0"/>
+        <origin xyz="0 -${wheel_separation / 2} -0.0538" rpy="${pi/2} 0 0"/>
         <axis xyz="0 0 -1"/>
         <limit effort="5.0" velocity="13.8"/>
