Commit message: Stabilize lidar navigation and safety

File: description/lidar.xacro (robot description, xacro)
@@ -4,5 +4,7 @@
         <parent link="chassis"/>
         <child link="laser_frame"/>
-        <origin xyz="0.91 0 0.082" rpy="0 0 0"/>
+        <!-- The drive axle is 0.15 m ahead of the chassis origin, placing
+             the measured lidar center 0.73 m ahead of the axle. -->
+        <origin xyz="0.88 0 0.082" rpy="0 0 0"/>
     </joint>
     <link name="laser_frame">
